File: hardware/KiCad/AVR_ISP_With_POGO_Pin.sch (KiCad schematic (older format))
At the start: 6 parts, among them P1 75869-131LF, P2 P50-B1

Commit message: Updates along newer Kicad version
Parts:
- D1: symbol library:Led_Small -> AVR_ISP_With_POGO_Pin-rescue:Led_Small-library
- P1: symbol library:CONN_02X03 -> AVR_ISP_With_POGO_Pin-rescue:CONN_02X03-library
- P2: symbol library:CONN_01X06 -> AVR_ISP_With_POGO_Pin-rescue:CONN_01X06-library
- S1: symbol library:Switch_SPST -> AVR_ISP_With_POGO_Pin-rescue:Switch_SPST-library
Changed lines of the file:
@@
 EESchema Schematic File Version 4
-LIBS:AVR_ISP_With_POGO_Pin-cache
 EELAYER 30 0
 EELAYER END
@@
 $EndDescr
 $Comp
-L library:CONN_01X06 P2
+L AVR_ISP_With_POGO_Pin-rescue:CONN_01X06-library P2
 U 1 1 587111A5
 P 7150 3000
@@
 $EndComp
 $Comp
-L library:CONN_02X03 P1
+L AVR_ISP_With_POGO_Pin-rescue:CONN_02X03-library P1
 U 1 1 587111D4
 P 4950 2950
@@
 $EndComp
 $Comp
-L library:Led_Small D1
+L AVR_ISP_With_POGO_Pin-rescue:Led_Small-library D1
 U 1 1 5871164C
 P 5100 4000
@@
 GND
 $Comp
-L library:Switch_SPST S1
+L AVR_ISP_With_POGO_Pin-rescue:Switch_SPST-library S1
 U 1 1 5871179A
 P 5000 4600
